File: cobra_keyboard.kicad_sch (KiCad schematic)
At the start: 93 parts

Commit message: Swap GRAPH and NEW MODE keys
Parts:
- CD1, CI1: value (none) -> 10uF; footprint (none) -> horizontal:CP_Radial_D4.0mm_P1.50mm_Horizontal
- D100, D101, D103, D104, D209, D301, D302, D501, D512: value (none) -> 1N4148; footprint (none) -> Diode_THT:D_DO-35_SOD27_P7.62mm_Horizontal
- H1, H2, H3, H4, H5, H6: value (none) -> MountingHole; footprint (none) -> MountingHole:MountingHole_3mm
- JKB1: value (none) -> Conn_02x10_Row_Letter_Last; footprint (none) -> Connector_PinHeader_2.54mm:PinHeader_2x10_P2.54mm_Vertical
- JLS1: value (none) -> Conn_01x02; footprint (none) -> Connector_PinHeader_2.54mm:PinHeader_1x02_P2.54mm_Vertical
- K100: value (none) -> DOWN; footprint (none) -> Button_Switch_Keyboard:SW_Cherry_MX_1.00u_PCB
- K101: value (none) -> UP; footprint (none) -> Button_Switch_Keyboard:SW_Cherry_MX_1.00u_PCB
- K102: value (none) -> SPACE; footprint (none) -> Button_Switch_Keyboard:SW_Cherry_MX_6.25u_PCB
- K103: value (none) -> LEFT; footprint (none) -> Button_Switch_Keyboard:SW_Cherry_MX_1.00u_PCB
- K104: value (none) -> RIGHT; footprint (none) -> Button_Switch_Keyboard:SW_Cherry_MX_1.00u_PCB
- K200: value (none) -> CTRL; footprint (none) -> Button_Switch_Keyboard:SW_Cherry_MX_1.00u_PCB
- K201: value (none) -> CS; footprint (none) -> Button_Switch_Keyboard:SW_Cherry_MX_2.25u_PCB
- K202: value (none) -> Z; footprint (none) -> Button_Switch_Keyboard:SW_Cherry_MX_1.00u_PCB
- K203: value (none) -> X; footprint (none) -> Button_Switch_Keyboard:SW_Cherry_MX_1.00u_PCB
- K204: value (none) -> C; footprint (none) -> Button_Switch_Keyboard:SW_Cherry_MX_1.00u_PCB
- K205: value (none) -> V; footprint (none) -> Button_Switch_Keyboard:SW_Cherry_MX_1.00u_PCB
- K206: value (none) -> B; footprint (none) -> Button_Switch_Keyboard:SW_Cherry_MX_1.00u_PCB
- K207: value (none) -> N; footprint (none) -> Button_Switch_Keyboard:SW_Cherry_MX_1.00u_PCB
- K208: value (none) -> M; footprint (none) -> Button_Switch_Keyboard:SW_Cherry_MX_1.00u_PCB
- K209: value (none) -> NEW M; footprint (none) -> Button_Switch_Keyboard:SW_Cherry_MX_1.00u_PCB
- K210: value (none) -> SS; footprint (none) -> Button_Switch_Keyboard:SW_Cherry_MX_2.75u_PCB
- K211: value (none) -> F4; footprint (none) -> Button_Switch_Keyboard:SW_Cherry_MX_1.00u_PCB
- K300: value (none) -> NO SCR; footprint (none) -> Button_Switch_Keyboard:SW_Cherry_MX_1.00u_PCB
- K301: value (none) -> CS LK; footprint (none) -> Button_Switch_Keyboard:SW_Cherry_MX_1.75u_PCB
- K302: value (none) -> GRAPH; footprint (none) -> Button_Switch_Keyboard:SW_Cherry_MX_1.50u_PCB
- K303: value (none) -> A; footprint (none) -> Button_Switch_Keyboard:SW_Cherry_MX_1.00u_PCB
- K304: value (none) -> S; footprint (none) -> Button_Switch_Keyboard:SW_Cherry_MX_1.00u_PCB
- K305: value (none) -> D; footprint (none) -> Button_Switch_Keyboard:SW_Cherry_MX_1.00u_PCB
- K306: value (none) -> F; footprint (none) -> Button_Switch_Keyboard:SW_Cherry_MX_1.00u_PCB
- K307: value (none) -> G; footprint (none) -> Button_Switch_Keyboard:SW_Cherry_MX_1.00u_PCB
- K308: value (none) -> H; footprint (none) -> Button_Switch_Keyboard:SW_Cherry_MX_1.00u_PCB
- K309: value (none) -> J; footprint (none) -> Button_Switch_Keyboard:SW_Cherry_MX_1.00u_PCB
- K310: value (none) -> K; footprint (none) -> Button_Switch_Keyboard:SW_Cherry_MX_1.00u_PCB
- K311: value (none) -> L; footprint (none) -> Button_Switch_Keyboard:SW_Cherry_MX_1.00u_PCB
- K312: value (none) -> ENTER; footprint (none) -> Button_Switch_Keyboard:SW_Cherry_MX_2.25u_PCB
- K313: value (none) -> F3; footprint (none) -> Button_Switch_Keyboard:SW_Cherry_MX_1.00u_PCB
- K400: value (none) -> LF; footprint (none) -> Button_Switch_Keyboard:SW_Cherry_MX_1.00u_PCB
- K401: value (none) -> TAB; footprint (none) -> Button_Switch_Keyboard:SW_Cherry_MX_1.50u_PCB
- K402: value (none) -> Q; footprint (none) -> Button_Switch_Keyboard:SW_Cherry_MX_1.00u_PCB
- K403: value (none) -> W; footprint (none) -> Button_Switch_Keyboard:SW_Cherry_MX_1.00u_PCB
- K404: value (none) -> E; footprint (none) -> Button_Switch_Keyboard:SW_Cherry_MX_1.00u_PCB
- K405: value (none) -> R; footprint (none) -> Button_Switch_Keyboard:SW_Cherry_MX_1.00u_PCB
- K406: value (none) -> T; footprint (none) -> Button_Switch_Keyboard:SW_Cherry_MX_1.00u_PCB
- K407: value (none) -> Y; footprint (none) -> Button_Switch_Keyboard:SW_Cherry_MX_1.00u_PCB
- K408: value (none) -> U; footprint (none) -> Button_Switch_Keyboard:SW_Cherry_MX_1.00u_PCB
- K409: value (none) -> I; footprint (none) -> Button_Switch_Keyboard:SW_Cherry_MX_1.00u_PCB
- K410: value (none) -> O; footprint (none) -> Button_Switch_Keyboard:SW_Cherry_MX_1.00u_PCB
- K411: value (none) -> P; footprint (none) -> Button_Switch_Keyboard:SW_Cherry_MX_1.00u_PCB
- K412: value (none) -> F2; footprint (none) -> Button_Switch_Keyboard:SW_Cherry_MX_1.00u_PCB
- K500: value (none) -> ESC; footprint (none) -> Button_Switch_Keyboard:SW_Cherry_MX_1.00u_PCB
- K501: value (none) -> PG ED; footprint (none) -> Button_Switch_Keyboard:SW_Cherry_MX_1.00u_PCB
- K502: value (none) -> 1; footprint (none) -> Button_Switch_Keyboard:SW_Cherry_MX_1.00u_PCB
- K503: value (none) -> 2; footprint (none) -> Button_Switch_Keyboard:SW_Cherry_MX_1.00u_PCB
- K504: value (none) -> 3; footprint (none) -> Button_Switch_Keyboard:SW_Cherry_MX_1.00u_PCB
- K505: value (none) -> 4; footprint (none) -> Button_Switch_Keyboard:SW_Cherry_MX_1.00u_PCB
- K506: value (none) -> 5; footprint (none) -> Button_Switch_Keyboard:SW_Cherry_MX_1.00u_PCB
- K507: value (none) -> 6; footprint (none) -> Button_Switch_Keyboard:SW_Cherry_MX_1.00u_PCB
- K508: value (none) -> 7; footprint (none) -> Button_Switch_Keyboard:SW_Cherry_MX_1.00u_PCB
- K509: value (none) -> 8; footprint (none) -> Button_Switch_Keyboard:SW_Cherry_MX_1.00u_PCB
- K510: value (none) -> 9; footprint (none) -> Button_Switch_Keyboard:SW_Cherry_MX_1.00u_PCB
- K511: value (none) -> 0; footprint (none) -> Button_Switch_Keyboard:SW_Cherry_MX_1.00u_PCB
- K512: value (none) -> DEL; footprint (none) -> Button_Switch_Keyboard:SW_Cherry_MX_2.00u_PCB
- K513: value (none) -> F1; footprint (none) -> Button_Switch_Keyboard:SW_Cherry_MX_1.00u_PCB
- R210, R411, RI1: value (none) -> 4.7K; footprint (none) -> Resistor_THT:R_Axial_DIN0204_L3.6mm_D1.6mm_P7.62mm_Horizontal
- RD1: value (none) -> 10K; footprint (none) -> Resistor_THT:R_Axial_DIN0204_L3.6mm_D1.6mm_P7.62mm_Horizontal
- RPU1: value (none) -> 1.5K; footprint (none) -> Resistor_THT:R_Axial_DIN0204_L3.6mm_D1.6mm_P7.62mm_Horizontal
- T201, T210, T411, T502, T503, T506, T507, T508, T509, T510, T511: value (none) -> BC337; footprint (none) -> horizontal:TO-92_Inline_Wide_Horizontal1
